Commit message: added realsense mount

File: urdf/arctos.urdf (robot description, URDF)
Before this commit: robot arctos, 11 links, 10 joints
Links:
- removed link tool
- added link realsense_mount; collision mesh filename=package://arctos_description/meshes/visual/realsense_mount.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; visual mesh filename=package://arctos_description/meshes/visual/realsense_mount.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
- added link tool0
- link left_jaw: geometry collision mesh filename=package://arctos_description/meshes/visual/left_jaw_v2.stl; visual mesh filename=package://arctos_description/meshes/visual/left_jaw_v2.stl
- link right_jaw: geometry collision mesh filename=package://arctos_description/meshes/visual/right_jaw_v2.stl; visual mesh filename=package://arctos_description/meshes/visual/right_jaw_v2.stl
Joints:
- removed joint gripper
- removed joint tool
- added joint link_6_to_mount: type fixed, parent link_6, child realsense_mount, origin xyz=0 0 0.006 rpy=0 0 0
- added joint mount_to_gripper: type fixed, parent realsense_mount, child gripper, origin xyz=0 0 0.003 rpy=0 0 0
- added joint tool0: type fixed, parent gripper, child tool0, origin xyz=0.0 0.0 0.13 rpy=0 0 0
- joint joint_1: limit lower=-3.14 upper=3.14 effort=87 velocity=2.3925 -> lower=-1.57 upper=1.57 effort=87 velocity=0.271765; origin xyz=0 0.00055605489707216942258 0.11100000143051147461 rpy=0 0 0 -> xyz=0 0.00055605489707216942258 0.1110 rpy=0 0 0
- joint joint_2: limit lower=-1.4 upper=2.2 effort=87 velocity=2.3925 -> lower=-0.524 upper=0.634 effort=87 velocity=0.026
- joint joint_3: limit lower=-1.6 upper=1.1 effort=87 velocity=2.3925 -> lower=-0.489 upper=0.341 effort=87 velocity=0.02321
- joint joint_4: limit lower=-3.14 upper=3.14 effort=87 velocity=2.3925 -> lower=-3.14 upper=3.14 effort=87 velocity=0.0763
- joint joint_5: limit lower=-1.8 upper=1.8 effort=87 velocity=2.3925 -> lower=-1.8 upper=1.8 effort=87 velocity=0.0543
- joint joint_6: limit lower=-3.14 upper=3.14 effort=87 velocity=2.3925 -> lower=-3.14 upper=3.14 effort=87 velocity=0.0543
- joint left_jaw: limit lower=0.0 upper=0.015 effort=87 velocity=2.3925 -> lower=0.0 upper=0.015 effort=87 velocity=0.1; origin xyz=0.0077708606105235935799 -0.030484645745930794014 0.039993524652900958039 rpy=1.570796326794896558 0 3.141592653589793116 -> xyz=-0.029515354775610149612 -0.011726639335887578675 0.039922151969763730595 rpy=1.570796326794896336 0 1.57079632679489678
- joint right_jaw: limit lower=0.0 upper=0.015 effort=87 velocity=2.3925 -> lower=0.0 upper=0.015 effort=87 velocity=0.1; origin xyz=-0.01172663933588792215 0.029515354775609847771 0.039922151969763619572 rpy=1.570796326794896558 0 0 -> xyz=0.030484645745930839117 0.0077708606105235666917 0.039993524652901180083 rpy=1.57079632679489678 0 -1.570796326794896558
